Commit message: Bugfixes

File: src/mobile_robot/model/robot.xacro (robot description, xacro)
@@ -1,7 +1,8 @@
+<?xml version="1.0" ?>
 <robot name="differential_drive_robot" xmlns:xacro="http://www.ros.org/wiki/xacro">
     <xacro:property name="pi_const" value="3.1415"/>
     <xacro:property name="a" value="1"/> <!-- Body-->
-    <xacro:property name="b" value="0.3"/> <!--Wheel-->
-    <xacro:property name="c" value="0.6"/> <!-- Chaste-->
+    <xacro:property name="b" value="0.3"/>
+    <xacro:property name="c" value="0.6"/>
     <!--Wheel-->
     <xacro:property name="r" value="0.15"/>
@@ -24,9 +25,9 @@
     <xacro:property name="I_wheel" value="${(1.0/12.0)*m2*(3.0*r*r+d*d)}"/>
     <xacro:property name="I_caster" value="${(2.0/5.0)*m3*r*r}"/>
-    <xacro:macro name="inertia_body">
+    <xacro:macro name="inertial_body">
         <inertial>
             <origin xyz="0.0 0.0 ${s1}" rpy="0.0 0.0 0.0"/>
             <mass value="${m1}"/>
-            <inertia ixx="${Ix_body}" ixy="0.0" ixz="0.0" iyy="Iy_body" iyz="0.0" izz="Iz_body"/>
+            <inertia ixx="${Ix_body}" ixy="0.0" ixz="0.0" iyy="${Iy_body}" iyz="0.0" izz="${Iz_body}"/>
         </inertial>
     </xacro:macro>
@@ -35,8 +36,8 @@
             <origin xyz="0.0 0.0 0.0" rpy="1.57075 0.0 0.0"/>
             <mass value="${m2}"/>
-            <inertia ixx="${I_wheel}" ixy="0.0" ixz="0.0" iyy="${Iy_wheel}" iyz="0.0" izz="${Iz_wheel}"/>
+            <inertia ixx="${I_wheel}" ixy="0.0" ixz="0.0" iyy="${I_wheel}" iyz="0.0" izz="${Iz_wheel}"/>
         </inertial>
     </xacro:macro>
-    <xacro:macro>
+    <xacro:macro name="inertial_chaste">
         <inertial>
             <origin xyz="0.0 0.0 0.0" rpy="0.0 0.0 0.0"/>
@@ -48,5 +49,5 @@
     <link name="base_footprint"></link>
     <joint name="body_link_joint" type="fixed">
-        <parent link="base_bootprint"/>
+        <parent link="base_footprint"/>
         <child link="body_link"/>
     </joint>
@@ -54,5 +55,5 @@
         <visual>
             <geometry>
-                <box size="${a} ${b} ${c}"/>
+                <box size="${a} ${c} ${b}"/>
             </geometry>
             <origin xyz="0.0 0.0 ${s1}" rpy="0 0 0"/>
@@ -66,8 +67,31 @@
         <xacro:inertial_body/>
     </link>
+    <joint name="caster_joint" type="revolute">
+        <parent link="body_link"/>
+        <child link="caster_link"/>
+        <origin xyz="${s3} ${0} ${r}"/>
+        <axis xyz="0 1 0"/>
+        <limit effort="50000.0" velocity="10.0"/>
+        <dynamics damping="1.0" friction="1.0"/>
+    </joint>
+    <link name="caster_link">
+        <visual>
+            <origin xyz="0.0 0.0 0.0" rpy="0 0.0 0.0"/>
+            <geometry>
+                <sphere radius="${r}"/>
+            </geometry>
+        </visual>
+        <collision>
+            <origin xyz="0.0 0.0 0.0" rpy="0 0.0 0.0"/>
+            <geometry>
+               <sphere radius="${r}"/>
+            </geometry>
+        </collision>
+        <xacro:inertial_chaste/>
+    </link>
     <joint name="wheel1_joint" type="continuous">
         <parent link="body_link"/>
         <child link="wheel1_link"/>
-        <origin xyz="${s2} ${-s4} ${r}"/>
+        <origin xyz="${-s2} ${-s4} ${r}"/>
         <axis xyz="0 1 0"/>
         <limit effort="50000.0" velocity="10.0"/>

Commit message: La til en rviz-fil og fiksa en bug i urdf-fila

File: src/mobile_robot/model/robot.xacro (robot description, xacro)
@@ -67,5 +67,5 @@
         <xacro:inertial_body/>
     </link>
-    <joint name="caster_joint" type="revolute">
+    <joint name="caster_joint" type="fixed">
         <parent link="body_link"/>
         <child link="caster_link"/>
